File: pcb/tartan.kicad_pcb (KiCad board)
At the start: 2 copper layers, 285 x 117 mm, 171 parts, among them J1 AVR_ISP_6, J2 USB_OTG, SW1 SW_Push, SW10 SW_Push, SW11 SW_Push, SW12 SW_Push, SW13 SW_Push, SW14 SW_Push, SW15 SW_Push, SW16 SW_Push, SW17 SW_Push, SW18 SW_Push, SW19 SW_Push, SW2 SW_Push, SW20 SW_Push, SW21 SW_Push, SW22 SW_Push, SW23 SW_Push, SW24 SW_Push, SW25 SW_Push, SW26 SW_Push, SW27 SW_Push, SW28 SW_Push, SW29 SW_Push, SW3 SW_Push, SW30 SW_Push, SW31 SW_Push, SW32 SW_Push, SW33 SW_Push, SW34 SW_Push, SW35 SW_Push, SW36 SW_Push, SW37 SW_Push, SW38 SW_Push, SW39 SW_Push, SW4 SW_Push, SW40 SW_Push, SW41 SW_Push, SW42 SW_Push, SW43 SW_Push, SW44 SW_Push, SW45 SW_Push, SW46 SW_Push, SW47 SW_Push, SW48 SW_Push, SW49 SW_Push, SW5 SW_Push, SW50 SW_Push, SW51 SW_Push, SW52 SW_Push, SW53 SW_Push, SW54 SW_Push, SW55 SW_Push, SW56 SW_Push, SW57 SW_Push, SW58 SW_Push, SW59 SW_Push, SW6 SW_Push, SW60 SW_Push, SW61 SW_Push, SW62 SW_Push, SW63 SW_Push, SW64 SW_Push, SW65 SW_Push, SW66 SW_Push, SW67 SW_Push, SW68 SW_Push, SW69 SW_Push, SW7 SW_Push, SW70 RESET, SW71 BOOT, SW8 SW_Push, SW9 SW_Push, U1 ATMEGA328-PU, Y1 16MHz

Commit message: Added new routing for matrix, still need to add USB C.
Parts:
- removed STAB1, STAB2, STAB3, STAB4, STAB5: 2U, SMKJP:Stab_MX_2u
- removed STAB6: 2U, Button_Switch_Keyboard:SW_Cherry_MX1A_6.25u_PCB
- C1: footprint Capacitors_THT:CP_Radial_D4.0mm_P1.50mm -> Capacitor_THT:CP_Radial_D4.0mm_P1.50mm
- C2, C3: footprint Capacitors_THT:C_Disc_D4.3mm_W1.9mm_P5.00mm -> Capacitor_THT:C_Disc_D4.3mm_W1.9mm_P5.00mm
- C4, C5: footprint Capacitors_THT:C_Disc_D3.0mm_W1.6mm_P2.50mm -> Capacitor_THT:C_Disc_D3.0mm_W1.6mm_P2.50mm
- D1, D10, D11, D12, D13, D14, D15, D16, D17, D18, D19, D2, D20, D21, D22, D23, D24, D25, D26, D27, D28, D29, D3, D30, D31, D32, D33, D34, D35, D36, D37, D38, D39, D4, D40, D41, D42, D43, D44, D45, D46, D47, D48, D49, D5, D50, D51, D52, D53, D54, D55, D56, D57, D58, D59, D6, D60, D61, D62, D63, D64, D65, D66, D7, D8, D9: footprint dm9_rc:D_DO-35_SOD27_P5.08mm_Horizontal -> tartan:D_DO-35_SOD27_P5.08mm_Horizontal
- F1: footprint dm9_miscs:polyfuse_5.1mm -> tartan:polyfuse_5.1mm
- H1, H10, H11, H2, H3, H4, H5, H6, H7, H8, H9: footprint Mounting_Holes:MountingHole_2.2mm_M2_Pad -> MountingHole:MountingHole_2.2mm_M2
- J1: footprint Pin_Headers:Pin_Header_Straight_2x03_Pitch2.54mm -> Connector_PinHeader_2.54mm:PinHeader_2x03_P2.54mm_Vertical
- J2: footprint dm9_conn:USB_MINIB_Akizuki_MUSB-5BF01AS -> tartan:USB_MINIB_Akizuki_MUSB-5BF01AS
- R1, R2, R3, R4: footprint Resistors_THT:R_Axial_DIN0204_L3.6mm_D1.6mm_P5.08mm_Horizontal -> Resistor_THT:R_Axial_DIN0204_L3.6mm_D1.6mm_P5.08mm_Horizontal
- SW66: footprint SMKJP:SW_Cherry_MX1A_1.50u_PCB -> tartan:Tartan_SW_Cherry_MX1A_1.50u_PCB
- SW70, SW71: footprint Buttons_Switches_THT:SW_PUSH_6mm -> Button_Switch_THT:SW_PUSH_6mm
- U1: footprint Housings_DIP:DIP-28_W7.62mm -> Package_DIP:DIP-28_W7.62mm
- Y1: footprint Crystals:Crystal_HC49-4H_Vertical -> Crystal:Crystal_HC49-4H_Vertical
Connections:
- C4 pad 1: Net-(C4-Pad1) -> Net-(U1-XTAL1/PB6)
- C5 pad 1: Net-(C5-Pad1) -> Net-(U1-XTAL2/PB7)
- J2 pad 4: (no net) -> unconnected-(J2-ID-Pad4)
- J2 pad 6: (no net) -> unconnected-(J2-Shield-Pad6)
- U1 pad 10: Net-(C4-Pad1) -> Net-(U1-XTAL2/PB7)
- U1 pad 21: (no net) -> unconnected-(U1-AREF-Pad21)
- U1 pad 9: Net-(C5-Pad1) -> Net-(U1-XTAL1/PB6)
- Y1 pad 1: Net-(C5-Pad1) -> Net-(U1-XTAL1/PB6)
- Y1 pad 2: Net-(C4-Pad1) -> Net-(U1-XTAL2/PB7)
Routing:
- net /ROW4: track 223.3 -> 254.0 mm, vias 0 -> 12
- net /ROW3: track 196.9 -> 224.7 mm, vias 0 -> 15
- net Net-(U1-XTAL1/PB6): track 0.00 -> 16.7 mm
- net Net-(U1-XTAL2/PB7): track 0.00 -> 15.6 mm
- net /ROW1: track 210.0 -> 223.4 mm, vias 0 -> 13
- net Net-(C4-Pad1): track 11.9 -> 0.00 mm
- net Net-(C5-Pad1): track 10.5 -> 0.00 mm
- net /ROW0: track 213.3 -> 206.2 mm
- net /ROW2: track 216.9 -> 211.2 mm, vias 0 -> 12
- net /COL11: track 129.0 -> 127.1 mm
- net Net-(D4-A): track 16.2 -> 15.7 mm
- net /USB_D-: track 6.13 -> 5.62 mm
- net GND: track 13.4 -> 13.1 mm, vias 67 -> 66
Other:
- net class Default removed
- board text added: "Tartan # Through Hole Rev.2 (c)2019 Takuya Urakawa, Dm9Records, 5z6p.com (c) Kim C, FUBAR Labs (for fun!)"
- board text removed: "Tartan # Through Hole Rev.1 (c)2019 Takuya Urakawa, Dm9Records, 5z6p.com"
