File: pcb/tartan.kicad_pcb (KiCad board)
At the start: 2 copper layers, 285 x 117 mm, 165 parts, among them J1 AVR_ISP_6, J2 USB_OTG, SW1 SW_Push, SW10 SW_Push, SW11 SW_Push, SW12 SW_Push, SW13 SW_Push, SW14 SW_Push, SW15 SW_Push, SW16 SW_Push, SW17 SW_Push, SW18 SW_Push, SW19 SW_Push, SW2 SW_Push, SW20 SW_Push, SW21 SW_Push, SW22 SW_Push, SW23 SW_Push, SW24 SW_Push, SW25 SW_Push, SW26 SW_Push, SW27 SW_Push, SW28 SW_Push, SW29 SW_Push, SW3 SW_Push, SW30 SW_Push, SW31 SW_Push, SW32 SW_Push, SW33 SW_Push, SW34 SW_Push, SW35 SW_Push, SW36 SW_Push, SW37 SW_Push, SW38 SW_Push, SW39 SW_Push, SW4 SW_Push, SW40 SW_Push, SW41 SW_Push, SW42 SW_Push, SW43 SW_Push, SW44 SW_Push, SW45 SW_Push, SW46 SW_Push, SW47 SW_Push, SW48 SW_Push, SW49 SW_Push, SW5 SW_Push, SW50 SW_Push, SW51 SW_Push, SW52 SW_Push, SW53 SW_Push, SW54 SW_Push, SW55 SW_Push, SW56 SW_Push, SW57 SW_Push, SW58 SW_Push, SW59 SW_Push, SW6 SW_Push, SW60 SW_Push, SW61 SW_Push, SW62 SW_Push, SW63 SW_Push, SW64 SW_Push, SW65 SW_Push, SW66 SW_Push, SW67 SW_Push, SW68 SW_Push, SW69 SW_Push, SW7 SW_Push, SW70 RESET, SW71 BOOT, SW8 SW_Push, SW9 SW_Push, U1 ATMEGA328-PU, Y1 16MHz

Commit message: Fix broken traces and too small vias... hopefully.
Parts:
- moved Y1 4.78 mm to (230.8, 35.8), turned to 0 degrees
Routing:
- net /ROW0: track 206.2 -> 224.1 mm
- net /ROW3: track 224.7 -> 210.8 mm, vias 15 -> 14
- net Net-(D60-A): track 121.8 -> 134.3 mm, vias 0 -> 1
- net /COL3: track 289.5 -> 300.7 mm
- net /COL1: track 263.2 -> 273.1 mm
- net /COL2: track 268.2 -> 277.3 mm
- net /COL9: track 166.8 -> 175.3 mm
- net /COL5: track 266.6 -> 273.3 mm
- net /COL6: track 275.1 -> 281.1 mm
- net Net-(U1-XTAL2/PB7): track 15.6 -> 9.83 mm
- net /ROW1: track 223.4 -> 217.7 mm, vias 13 -> 1
- net /COL12: track 122.0 -> 126.9 mm
- net /COL7: track 282.2 -> 286.4 mm
- net /COL11: track 127.1 -> 131.0 mm
- net GND: track 13.1 -> 9.56 mm, vias 66 -> 37
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Other:
- board text added: "VCC"
- board text removed: "+5V"

Commit message: Updated to use new footprints, removed backups directory, as well as specifically removed bottom PCB for sanity savings.
Parts:
- removed G***: LOGO, tartan:band
- removed G***: LOGO, tartan:logo1
- added J3: Conn_01x01_Pin, tartan:bottom1_mask, B.Cu at (169.0, 102.5)
- moved C3 3.88 mm to (234.4, 50.3)
Routing:
- net Net-(D60-A): track 134.3 -> 117.1 mm
- net /COL4: track 275.4 -> 281.8 mm
- net Net-(D53-A): track 140.0 -> 146.4 mm
- net /COL2: track 277.3 -> 273.2 mm
- net /COL6: track 281.1 -> 285.1 mm
- net Net-(D3-A): track 16.9 -> 20.2 mm
- net /COL10: track 160.4 -> 163.6 mm
- net /COL7: track 286.4 -> 289.3 mm
- net GND: track 9.56 -> 7.10 mm, vias 37 -> 33
- net +5V: track 116.2 -> 118.6 mm
- net /ROW4: track 252.8 -> 251.4 mm
- net /COL11: track 131.0 -> 132.5 mm
- net /COL8: track 132.5 -> 133.4 mm
- net /COL12: track 126.9 -> 127.8 mm
- net Net-(D65-K): track 16.2 -> 15.5 mm
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Other:
- rule pad_to_mask_clearance: 0.051 -> 0

Commit message: Little thing called broken traces updated.  Rounded some more too I guess.
Parts:
- moved J3 13.3 mm to (182.1, 100.2)
Routing:
- net /COL11: track 132.5 -> 125.3 mm
- net /ROW2: track 209.9 -> 206.9 mm
- net +5V: track 118.6 -> 116.6 mm
- net /COL9: track 174.6 -> 172.8 mm
- net /ROW0: track 224.1 -> 222.5 mm
- net /COL12: track 127.8 -> 126.4 mm
- net /ROW1: track 217.5 -> 216.4 mm
- net Net-(D64-A): track 201.9 -> 201.1 mm
- net Net-(D15-A): track 132.5 -> 131.7 mm
- net Net-(D24-A): track 44.2 -> 43.5 mm
- net /COL2: track 273.2 -> 273.9 mm
- net Net-(D47-A): track 88.0 -> 87.4 mm
- net Net-(D61-A): track 155.0 -> 154.4 mm
- net /COL3: track 300.1 -> 299.5 mm
- net Net-(D63-A): track 180.7 -> 180.2 mm
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