File: pcb/tartan.kicad_pcb (KiCad board)
At the start: 2 copper layers, 285 x 117 mm, 164 parts, among them J1 AVR_ISP_6, J2 USB_OTG, J3 Conn_01x01_Pin, SW1 SW_Push, SW10 SW_Push, SW11 SW_Push, SW12 SW_Push, SW13 SW_Push, SW14 SW_Push, SW15 SW_Push, SW16 SW_Push, SW17 SW_Push, SW18 SW_Push, SW19 SW_Push, SW2 SW_Push, SW20 SW_Push, SW21 SW_Push, SW22 SW_Push, SW23 SW_Push, SW24 SW_Push, SW25 SW_Push, SW26 SW_Push, SW27 SW_Push, SW28 SW_Push, SW29 SW_Push, SW3 SW_Push, SW30 SW_Push, SW31 SW_Push, SW32 SW_Push, SW33 SW_Push, SW34 SW_Push, SW35 SW_Push, SW36 SW_Push, SW37 SW_Push, SW38 SW_Push, SW39 SW_Push, SW4 SW_Push, SW40 SW_Push, SW41 SW_Push, SW42 SW_Push, SW43 SW_Push, SW44 SW_Push, SW45 SW_Push, SW46 SW_Push, SW47 SW_Push, SW48 SW_Push, SW49 SW_Push, SW5 SW_Push, SW50 SW_Push, SW51 SW_Push, SW52 SW_Push, SW53 SW_Push, SW54 SW_Push, SW55 SW_Push, SW56 SW_Push, SW57 SW_Push, SW58 SW_Push, SW59 SW_Push, SW6 SW_Push, SW60 SW_Push, SW61 SW_Push, SW62 SW_Push, SW63 SW_Push, SW64 SW_Push, SW65 SW_Push, SW66 SW_Push, SW67 SW_Push, SW68 SW_Push, SW69 SW_Push, SW7 SW_Push, SW70 RESET, SW71 BOOT, SW8 SW_Push, SW9 SW_Push, U1 ATMEGA328-PU, Y1 16MHz

Commit message: Rounded traces and re-added silks.  Oops.
Parts:
- added G***: LOGO, tartan:band, F.Cu at (107.1, 34.2)
Routing:
- net /COL8: track 133.1 -> 138.6 mm
- net Net-(D47-A): track 87.4 -> 90.0 mm
- net Net-(D54-A): track 145.4 -> 144.2 mm
- net /COL2: track 273.9 -> 272.6 mm
- net Net-(D51-A): track 118.6 -> 117.4 mm
- net Net-(D61-A): track 154.4 -> 153.2 mm
- net Net-(D63-A): track 180.2 -> 179.0 mm
- net Net-(D37-A): track 97.1 -> 96.0 mm
- net Net-(D62-A): track 167.1 -> 166.0 mm
- net Net-(D39-A): track 116.7 -> 115.6 mm
- net Net-(D50-A): track 105.3 -> 104.3 mm
- net Net-(D53-A): track 146.3 -> 145.2 mm
- net Net-(D55-A): track 172.5 -> 171.5 mm
- net Net-(D40-A): track 122.9 -> 122.0 mm
- net Net-(D38-A): track 102.7 -> 101.7 mm
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
Commit message: Small cleanup in latest nightly to hopefully minimize truly broken traces.
Routing:
- net /COL3: track 300.0 -> 304.4 mm
- net Net-(D51-A): track 117.4 -> 118.5 mm
- net Net-(D56-A): track 179.5 -> 180.2 mm
- net Net-(D60-A): vias 1 -> 0

Commit message: Update to new USB B that Ben found.
	new file:   pcb/sym-lib-table
Parts:
- removed J2: USB_OTG, tartan:USB_MINIB_Akizuki_MUSB-5BF01AS
- added J4: USB_OTG, tartan:USB B THT 1734510-1_TEC, F.Cu at (266.6, 35.0)
Routing:
- net GND: track 7.10 -> 2.54 mm, vias 43 -> 51
- net Net-(D66-K): track 18.4 -> 19.5 mm
- net /COL8: track 138.6 -> 137.5 mm
- net /COL5: track 273.5 -> 272.6 mm
- net Net-(D65-K): track 15.3 -> 16.1 mm
- net /COL11: track 125.3 -> 124.5 mm
- net /COL3: track 304.4 -> 303.8 mm
