File: pcb/tartan_bottom.kicad_pcb (KiCad board)
At the start: 2 copper layers, 285 x 117 mm, 17 parts

Commit message: Fix broken traces and too small vias... hopefully.
Other:
- net class Default removed
